Commit message: several fixes, working without dynamics and stpbv

File: romeo_description/urdf/romeo.urdf (robot description, URDF)
Before this commit: robot RomeoH37, 96 links, 95 joints
Links:
- removed link ImuTorsoAccelerometer_frame
- added link Accelerometer
Joints:
- joint AccelerometerDownTorso_sensor_fixedjoint: child ImuTorsoAccelerometer_frame -> Accelerometer

Commit message: fix more params, but still not working for dynamics/contact constraint

File: romeo_description/urdf/romeo.urdf (robot description, URDF)
Before this commit: robot RomeoH37, 96 links, 95 joints
Joints:
- joint LEyePitch: limit lower=-0.349066 upper=0.349066 effort=0.01752 velocity=293.215 -> lower=-0.349066 upper=0.349066 effort=0.01752 velocity=0.293215
- joint LEyeYaw: limit lower=-0.523599 upper=0.523599 effort=0.01752 velocity=293.215 -> lower=-0.523599 upper=0.523599 effort=0.01752 velocity=0.293215
- joint REyePitch: limit lower=-0.349066 upper=0.349066 effort=0.01752 velocity=293.215 -> lower=-0.349066 upper=0.349066 effort=0.01752 velocity=0.293215
- joint REyeYaw: limit lower=-0.523599 upper=0.523599 effort=0.01752 velocity=293.215 -> lower=-0.523599 upper=0.523599 effort=0.01752 velocity=0.293215
