Commit message: Changed pkg name from romeo_description to romeo_description_mc. Modified Xacro file for compatibility with multi contact.

File: romeo_description_mc/urdf/romeo.urdf (robot description, URDF)
Before this commit: robot RomeoH37, 96 links, 95 joints
Links:
- link Cap: geometry visual mesh filename=package://romeo_description_mc/meshes/Cap.dae scale=1 1 1
- link HeadRoll_link: geometry collision mesh filename=package://romeo_description_mc/meshes/HeadRoll_0.10.stl scale=1 1 1; visual mesh filename=package://romeo_description_mc/meshes/HeadRoll.dae scale=1 1 1
- link LElbow: geometry collision mesh filename=package://romeo_description_mc/meshes/LElbowYaw_0.10.stl scale=1 1 1; visual mesh filename=package://romeo_description_mc/meshes/LElbowYaw.dae scale=1 1 1
- link LEye: geometry collision mesh filename=package://romeo_description_mc/meshes/LEyePitch_0.10.stl scale=1 1 1; visual mesh filename=package://romeo_description_mc/meshes/LEyePitch.dae scale=1 1 1
- link LFinger11_link: geometry collision mesh filename=package://romeo_description_mc/meshes/LFinger11_0.10.stl scale=1 1 1; visual mesh filename=package://romeo_description_mc/meshes/LFinger11.dae scale=1 1 1
- link LFinger12_link: geometry collision mesh filename=package://romeo_description_mc/meshes/LFinger12_0.10.stl scale=1 1 1; visual mesh filename=package://romeo_description_mc/meshes/LFinger12.dae scale=1 1 1
- link LFinger13_link: geometry collision mesh filename=package://romeo_description_mc/meshes/LFinger13_0.10.stl scale=1 1 1; visual mesh filename=package://romeo_description_mc/meshes/LFinger13.dae scale=1 1 1
- link LFinger21_link: geometry collision mesh filename=package://romeo_description_mc/meshes/LFinger21_0.10.stl scale=1 1 1; visual mesh filename=package://romeo_description_mc/meshes/LFinger21.dae scale=1 1 1
- link LFinger22_link: geometry collision mesh filename=package://romeo_description_mc/meshes/LFinger22_0.10.stl scale=1 1 1; visual mesh filename=package://romeo_description_mc/meshes/LFinger22.dae scale=1 1 1
- link LFinger23_link: geometry collision mesh filename=package://romeo_description_mc/meshes/LFinger23_0.10.stl scale=1 1 1; visual mesh filename=package://romeo_description_mc/meshes/LFinger23.dae scale=1 1 1
- link LFinger31_link: geometry collision mesh filename=package://romeo_description_mc/meshes/LFinger31_0.10.stl scale=1 1 1; visual mesh filename=package://romeo_description_mc/meshes/LFinger31.dae scale=1 1 1
- link LFinger32_link: geometry collision mesh filename=package://romeo_description_mc/meshes/LFinger32_0.10.stl scale=1 1 1; visual mesh filename=package://romeo_description_mc/meshes/LFinger32.dae scale=1 1 1
- link LFinger33_link: geometry collision mesh filename=package://romeo_description_mc/meshes/LFinger33_0.10.stl scale=1 1 1; visual mesh filename=package://romeo_description_mc/meshes/LFinger33.dae scale=1 1 1
- link LShoulderYaw_link: geometry collision mesh filename=package://romeo_description_mc/meshes/LShoulderYaw_0.10.stl scale=1 1 1; visual mesh filename=package://romeo_description_mc/meshes/LShoulderYaw.dae scale=1 1 1
- link LThigh: geometry collision mesh filename=package://romeo_description_mc/meshes/LHipPitch_0.10.stl scale=1 1 1; visual mesh filename=package://romeo_description_mc/meshes/LHipPitch.dae scale=1 1 1
- link LThumb1_link: geometry collision mesh filename=package://romeo_description_mc/meshes/LThumb1_0.10.stl scale=1 1 1; visual mesh filename=package://romeo_description_mc/meshes/LThumb1.dae scale=1 1 1
- link LThumb2_link: geometry collision mesh filename=package://romeo_description_mc/meshes/LThumb2_0.10.stl scale=1 1 1; visual mesh filename=package://romeo_description_mc/meshes/LThumb2.dae scale=1 1 1
- link LThumb3_link: geometry collision mesh filename=package://romeo_description_mc/meshes/LThumb3_0.10.stl scale=1 1 1; visual mesh filename=package://romeo_description_mc/meshes/LThumb3.dae scale=1 1 1
- link LTibia: geometry collision mesh filename=package://romeo_description_mc/meshes/LKneePitch_0.10.stl scale=1 1 1; visual mesh filename=package://romeo_description_mc/meshes/LKneePitch.dae scale=1 1 1
- link LWristRoll_link: geometry collision mesh filename=package://romeo_description_mc/meshes/LWristRoll_0.10.stl scale=1 1 1; visual mesh filename=package://romeo_description_mc/meshes/LWristRoll.dae scale=1 1 1
- link LWristYaw_link: geometry collision mesh filename=package://romeo_description_mc/meshes/LWristYaw_0.10.stl scale=1 1 1; visual mesh filename=package://romeo_description_mc/meshes/LWristYaw.dae scale=1 1 1
- link NeckPitch_link: geometry collision mesh filename=package://romeo_description_mc/meshes/NeckPitch_0.10.stl scale=1 1 1; visual mesh filename=package://romeo_description_mc/meshes/NeckPitch.dae scale=1 1 1
- link RElbow: geometry collision mesh filename=package://romeo_description_mc/meshes/RElbowYaw_0.10.stl scale=1 1 1; visual mesh filename=package://romeo_description_mc/meshes/RElbowYaw.dae scale=1 1 1
- link REye: geometry collision mesh filename=package://romeo_description_mc/meshes/REyePitch_0.10.stl scale=1 1 1; visual mesh filename=package://romeo_description_mc/meshes/REyePitch.dae scale=1 1 1
- link RFinger11_link: geometry collision mesh filename=package://romeo_description_mc/meshes/RFinger11_0.10.stl scale=1 1 1; visual mesh filename=package://romeo_description_mc/meshes/RFinger11.dae scale=1 1 1
- link RFinger12_link: geometry collision mesh filename=package://romeo_description_mc/meshes/RFinger12_0.10.stl scale=1 1 1; visual mesh filename=package://romeo_description_mc/meshes/RFinger12.dae scale=1 1 1
- link RFinger13_link: geometry collision mesh filename=package://romeo_description_mc/meshes/RFinger13_0.10.stl scale=1 1 1; visual mesh filename=package://romeo_description_mc/meshes/RFinger13.dae scale=1 1 1
- link RFinger21_link: geometry collision mesh filename=package://romeo_description_mc/meshes/RFinger21_0.10.stl scale=1 1 1; visual mesh filename=package://romeo_description_mc/meshes/RFinger21.dae scale=1 1 1
- link RFinger22_link: geometry collision mesh filename=package://romeo_description_mc/meshes/RFinger22_0.10.stl scale=1 1 1; visual mesh filename=package://romeo_description_mc/meshes/RFinger22.dae scale=1 1 1
- link RFinger23_link: geometry collision mesh filename=package://romeo_description_mc/meshes/RFinger23_0.10.stl scale=1 1 1; visual mesh filename=package://romeo_description_mc/meshes/RFinger23.dae scale=1 1 1
- link RFinger31_link: geometry collision mesh filename=package://romeo_description_mc/meshes/RFinger31_0.10.stl scale=1 1 1; visual mesh filename=package://romeo_description_mc/meshes/RFinger31.dae scale=1 1 1
- link RFinger32_link: geometry collision mesh filename=package://romeo_description_mc/meshes/RFinger32_0.10.stl scale=1 1 1; visual mesh filename=package://romeo_description_mc/meshes/RFinger32.dae scale=1 1 1
- link RFinger33_link: geometry collision mesh filename=package://romeo_description_mc/meshes/RFinger33_0.10.stl scale=1 1 1; visual mesh filename=package://romeo_description_mc/meshes/RFinger33.dae scale=1 1 1
- link RShoulderYaw_link: geometry collision mesh filename=package://romeo_description_mc/meshes/RShoulderYaw_0.10.stl scale=1 1 1; visual mesh filename=package://romeo_description_mc/meshes/RShoulderYaw.dae scale=1 1 1
- link RThigh: geometry collision mesh filename=package://romeo_description_mc/meshes/RHipPitch_0.10.stl scale=1 1 1; visual mesh filename=package://romeo_description_mc/meshes/RHipPitch.dae scale=1 1 1
- link RThumb1_link: geometry collision mesh filename=package://romeo_description_mc/meshes/RThumb1_0.10.stl scale=1 1 1; visual mesh filename=package://romeo_description_mc/meshes/RThumb1.dae scale=1 1 1
- link RThumb2_link: geometry collision mesh filename=package://romeo_description_mc/meshes/RThumb2_0.10.stl scale=1 1 1; visual mesh filename=package://romeo_description_mc/meshes/RThumb2.dae scale=1 1 1
- link RThumb3_link: geometry collision mesh filename=package://romeo_description_mc/meshes/RThumb3_0.10.stl scale=1 1 1; visual mesh filename=package://romeo_description_mc/meshes/RThumb3.dae scale=1 1 1
- link RTibia: geometry collision mesh filename=package://romeo_description_mc/meshes/RKneePitch_0.10.stl scale=1 1 1; visual mesh filename=package://romeo_description_mc/meshes/RKneePitch.dae scale=1 1 1
- link RWristRoll_link: geometry collision mesh filename=package://romeo_description_mc/meshes/RWristRoll_0.10.stl scale=1 1 1; visual mesh filename=package://romeo_description_mc/meshes/RWristRoll.dae scale=1 1 1
- link RWristYaw_link: geometry collision mesh filename=package://romeo_description_mc/meshes/RWristYaw_0.10.stl scale=1 1 1; visual mesh filename=package://romeo_description_mc/meshes/RWristYaw.dae scale=1 1 1
- link body: geometry collision mesh filename=package://romeo_description_mc/meshes/TrunkYaw_0.10.stl scale=1 1 1; visual mesh filename=package://romeo_description_mc/meshes/TrunkYaw.dae scale=1 1 1
- link l_ankle: geometry collision mesh filename=package://romeo_description_mc/meshes/LAnkleRoll_0.10.stl scale=1 1 1; visual mesh filename=package://romeo_description_mc/meshes/LAnkleRoll.dae scale=1 1 1
- link l_wrist: geometry collision mesh filename=package://romeo_description_mc/meshes/LWristPitch_0.10.stl scale=1 1 1; visual mesh filename=package://romeo_description_mc/meshes/LWristPitch.dae scale=1 1 1
- link r_ankle: geometry collision mesh filename=package://romeo_description_mc/meshes/RAnkleRoll_0.10.stl scale=1 1 1; visual mesh filename=package://romeo_description_mc/meshes/RAnkleRoll.dae scale=1 1 1
- link r_wrist: geometry collision mesh filename=package://romeo_description_mc/meshes/RWristPitch_0.10.stl scale=1 1 1; visual mesh filename=package://romeo_description_mc/meshes/RWristPitch.dae scale=1 1 1
- link torso: geometry collision mesh filename=package://romeo_description_mc/meshes/Torso_0.10.stl scale=1 1 1; visual mesh filename=package://romeo_description_mc/meshes/Torso.dae scale=1 1 1
Joints:
- joint LEyePitch: limit lower=-0.349066 upper=0.349066 effort=0.01752 velocity=0.293215 -> lower=-0.349066 upper=0.349066 effort=0.01752 velocity=293.215
- joint LEyeYaw: limit lower=-0.523599 upper=0.523599 effort=0.01752 velocity=0.293215 -> lower=-0.523599 upper=0.523599 effort=0.01752 velocity=293.215
- joint REyePitch: limit lower=-0.349066 upper=0.349066 effort=0.01752 velocity=0.293215 -> lower=-0.349066 upper=0.349066 effort=0.01752 velocity=293.215
- joint REyeYaw: limit lower=-0.523599 upper=0.523599 effort=0.01752 velocity=0.293215 -> lower=-0.523599 upper=0.523599 effort=0.01752 velocity=293.215

File: romeo_description_mc/urdf/romeo_cap.xacro (robot description, xacro)
@@ -22,5 +22,5 @@
       <visual>
         <geometry>
-          <mesh filename="package://romeo_description/meshes/Cap.dae" scale="1 1 1"/>
+          <mesh filename="package://romeo_description_mc/meshes/Cap.dae" scale="1 1 1"/>
         </geometry>
         <origin rpy="0 0 0" xyz="0 0 0"/>

File: romeo_description_mc/urdf/romeo_head.xacro (robot description, xacro)
@@ -4,4 +4,11 @@
  *********************************************************************-->
 <robot xmlns:xacro="http://www.ros.org/wiki/xacro">
+	<link name="base_link"/>
+	<joint name="base_link_fixedjoint" type="fixed">
+		<parent link="base_link"/>
+		<child link="torso"/>
+		<origin rpy="0 0 0" xyz="0 0 0"/>
+		<axis xyz="0 0 0"/>
+	</joint>
 	<joint name="NeckYaw" type="revolute">
 		<parent link="torso"/>

File: romeo_description_mc/urdf/romeo_sensors.xacro (robot description, xacro)
@@ -176,8 +176,10 @@
 		<axis xyz="0 0 0"/>
 	</joint>
-	<link name="ImuTorsoAccelerometer_frame"/>
+	<!--   <link name="ImuTorsoAccelerometer_frame"/> -->
+    <link name="Accelerometer"/>
 	<joint name="AccelerometerDownTorso_sensor_fixedjoint" type="fixed">
 		<parent link="body"/>
-		<child link="ImuTorsoAccelerometer_frame"/>
+		<!--     <child link="ImuTorsoAccelerometer_frame"/> -->
+        <child link="Accelerometer"/> <!--FIXME: see link definition-->
 		<origin rpy="0 0 0" xyz="0.06185 0.0087 -0.1582"/>
 		<axis xyz="0 0 0"/>

File: romeo_description_mc/urdf/romeo_torso.xacro (robot description, xacro)
@@ -4,5 +4,5 @@
  *********************************************************************-->
 <robot xmlns:xacro="http://www.ros.org/wiki/xacro">
-	<link name="base_link"/>
+	<!--link name="base_link"/>
 	<joint name="base_link_fixedjoint" type="fixed">
 		<parent link="base_link"/>
@@ -10,5 +10,5 @@
 		<origin rpy="0 0 0" xyz="0 0 0"/>
 		<axis xyz="0 0 0"/>
-	</joint>
+	</joint-->
 	<link name="torso">
 		<inertial>
