Commit message: Changed pkg name from romeo_description to romeo_description_mc. Modified Xacro file for compatibility with multi contact.

File: romeo_description_mc/urdf/romeo_visual_collisions.xacro (robot description, xacro)
@@ -7,11 +7,11 @@
 		<visual>
 			<geometry>
-				<mesh filename="package://romeo_description/meshes/REyePitch.dae" scale="1 1 1"/>
-			</geometry>
-			<origin rpy="0 0 0" xyz="0 0 0"/>
-		</visual>
-		<collision>
-			<geometry>
-				<mesh filename="package://romeo_description/meshes/REyePitch_0.10.stl" scale="1 1 1"/>
+				<mesh filename="package://romeo_description_mc/meshes/REyePitch.dae" scale="1 1 1"/>
+			</geometry>
+			<origin rpy="0 0 0" xyz="0 0 0"/>
+		</visual>
+		<collision>
+			<geometry>
+				<mesh filename="package://romeo_description_mc/meshes/REyePitch_0.10.stl" scale="1 1 1"/>
 			</geometry>
 			<origin rpy="0 0 0" xyz="0 0 0"/>
@@ -21,11 +21,11 @@
 		<visual>
 			<geometry>
-				<mesh filename="package://romeo_description/meshes/RFinger13.dae" scale="1 1 1"/>
-			</geometry>
-			<origin rpy="0 0 0" xyz="0 0 0"/>
-		</visual>
-		<collision>
-			<geometry>
-				<mesh filename="package://romeo_description/meshes/RFinger13_0.10.stl" scale="1 1 1"/>
+				<mesh filename="package://romeo_description_mc/meshes/RFinger13.dae" scale="1 1 1"/>
+			</geometry>
+			<origin rpy="0 0 0" xyz="0 0 0"/>
+		</visual>
+		<collision>
+			<geometry>
+				<mesh filename="package://romeo_description_mc/meshes/RFinger13_0.10.stl" scale="1 1 1"/>
 			</geometry>
 			<origin rpy="0 0 0" xyz="0 0 0"/>
@@ -35,11 +35,11 @@
 		<visual>
 			<geometry>
-				<mesh filename="package://romeo_description/meshes/RHipPitch.dae" scale="1 1 1"/>
-			</geometry>
-			<origin rpy="0 0 0" xyz="0 0 0"/>
-		</visual>
-		<collision>
-			<geometry>
-				<mesh filename="package://romeo_description/meshes/RHipPitch_0.10.stl" scale="1 1 1"/>
+				<mesh filename="package://romeo_description_mc/meshes/RHipPitch.dae" scale="1 1 1"/>
+			</geometry>
+			<origin rpy="0 0 0" xyz="0 0 0"/>
+		</visual>
+		<collision>
+			<geometry>
+				<mesh filename="package://romeo_description_mc/meshes/RHipPitch_0.10.stl" scale="1 1 1"/>
 			</geometry>
 			<origin rpy="0 0 0" xyz="0 0 0"/>
@@ -49,11 +49,11 @@
 		<visual>
 			<geometry>
-				<mesh filename="package://romeo_description/meshes/RFinger12.dae" scale="1 1 1"/>
-			</geometry>
-			<origin rpy="0 0 0" xyz="0 0 0"/>
-		</visual>
-		<collision>
-			<geometry>
-				<mesh filename="package://romeo_description/meshes/RFinger12_0.10.stl" scale="1 1 1"/>
+				<mesh filename="package://romeo_description_mc/meshes/RFinger12.dae" scale="1 1 1"/>
+			</geometry>
+			<origin rpy="0 0 0" xyz="0 0 0"/>
+		</visual>
+		<collision>
+			<geometry>
+				<mesh filename="package://romeo_description_mc/meshes/RFinger12_0.10.stl" scale="1 1 1"/>
 			</geometry>
 			<origin rpy="0 0 0" xyz="0 0 0"/>
@@ -63,11 +63,11 @@
 		<visual>
 			<geometry>
-				<mesh filename="package://romeo_description/meshes/LFinger33.dae" scale="1 1 1"/>
-			</geometry>
-			<origin rpy="0 0 0" xyz="0 0 0"/>
-		</visual>
-		<collision>
-			<geometry>
-				<mesh filename="package://romeo_description/meshes/LFinger33_0.10.stl" scale="1 1 1"/>
+				<mesh filename="package://romeo_description_mc/meshes/LFinger33.dae" scale="1 1 1"/>
+			</geometry>
+			<origin rpy="0 0 0" xyz="0 0 0"/>
+		</visual>
+		<collision>
+			<geometry>
+				<mesh filename="package://romeo_description_mc/meshes/LFinger33_0.10.stl" scale="1 1 1"/>
 			</geometry>
 			<origin rpy="0 0 0" xyz="0 0 0"/>
@@ -77,11 +77,11 @@
 		<visual>
 			<geometry>
-				<mesh filename="package://romeo_description/meshes/RFinger31.dae" scale="1 1 1"/>
-			</geometry>
-			<origin rpy="0 0 0" xyz="0 0 0"/>
-		</visual>
-		<collision>
-			<geometry>
-				<mesh filename="package://romeo_description/meshes/RFinger31_0.10.stl" scale="1 1 1"/>
+				<mesh filename="package://romeo_description_mc/meshes/RFinger31.dae" scale="1 1 1"/>
+			</geometry>
+			<origin rpy="0 0 0" xyz="0 0 0"/>
+		</visual>
+		<collision>
+			<geometry>
+				<mesh filename="package://romeo_description_mc/meshes/RFinger31_0.10.stl" scale="1 1 1"/>
 			</geometry>
 			<origin rpy="0 0 0" xyz="0 0 0"/>
@@ -91,11 +91,11 @@
 		<visual>
 			<geometry>
-				<mesh filename="package://romeo_description/meshes/LWristYaw.dae" scale="1 1 1"/>
-			</geometry>
-			<origin rpy="0 0 0" xyz="0 0 0"/>
-		</visual>
-		<collision>
-			<geometry>
-				<mesh filename="package://romeo_description/meshes/LWristYaw_0.10.stl" scale="1 1 1"/>
+				<mesh filename="package://romeo_description_mc/meshes/LWristYaw.dae" scale="1 1 1"/>
+			</geometry>
+			<origin rpy="0 0 0" xyz="0 0 0"/>
+		</visual>
+		<collision>
+			<geometry>
+				<mesh filename="package://romeo_description_mc/meshes/LWristYaw_0.10.stl" scale="1 1 1"/>
 			</geometry>
 			<origin rpy="0 0 0" xyz="0 0 0"/>
@@ -105,11 +105,11 @@
 		<visual>
 			<geometry>
-				<mesh filename="package://romeo_description/meshes/RFinger32.dae" scale="1 1 1"/>
-			</geometry>
-			<origin rpy="0 0 0" xyz="0 0 0"/>
-		</visual>
-		<collision>
-			<geometry>
-				<mesh filename="package://romeo_description/meshes/RFinger32_0.10.stl" scale="1 1 1"/>
+				<mesh filename="package://romeo_description_mc/meshes/RFinger32.dae" scale="1 1 1"/>
+			</geometry>
+			<origin rpy="0 0 0" xyz="0 0 0"/>
+		</visual>
+		<collision>
+			<geometry>
+				<mesh filename="package://romeo_description_mc/meshes/RFinger32_0.10.stl" scale="1 1 1"/>
 			</geometry>
 			<origin rpy="0 0 0" xyz="0 0 0"/>
@@ -119,11 +119,11 @@
 		<visual>
 			<geometry>
-				<mesh filename="package://romeo_description/meshes/LFinger21.dae" scale="1 1 1"/>
-			</geometry>
-			<origin rpy="0 0 0" xyz="0 0 0"/>
-		</visual>
-		<collision>
-			<geometry>
-				<mesh filename="package://romeo_description/meshes/LFinger21_0.10.stl" scale="1 1 1"/>
+				<mesh filename="package://romeo_description_mc/meshes/LFinger21.dae" scale="1 1 1"/>
+			</geometry>
+			<origin rpy="0 0 0" xyz="0 0 0"/>
+		</visual>
+		<collision>
+			<geometry>
+				<mesh filename="package://romeo_description_mc/meshes/LFinger21_0.10.stl" scale="1 1 1"/>
 			</geometry>
 			<origin rpy="0 0 0" xyz="0 0 0"/>
@@ -133,11 +133,11 @@
 		<visual>
 			<geometry>
-				<mesh filename="package://romeo_description/meshes/LFinger13.dae" scale="1 1 1"/>
-			</geometry>
-			<origin rpy="0 0 0" xyz="0 0 0"/>
-		</visual>
-		<collision>
-			<geometry>
-				<mesh filename="package://romeo_description/meshes/LFinger13_0.10.stl" scale="1 1 1"/>
+				<mesh filename="package://romeo_description_mc/meshes/LFinger13.dae" scale="1 1 1"/>
+			</geometry>
+			<origin rpy="0 0 0" xyz="0 0 0"/>
+		</visual>
+		<collision>
+			<geometry>
+				<mesh filename="package://romeo_description_mc/meshes/LFinger13_0.10.stl" scale="1 1 1"/>
 			</geometry>
 			<origin rpy="0 0 0" xyz="0 0 0"/>
@@ -147,11 +147,11 @@
 		<visual>
 			<geometry>
-				<mesh filename="package://romeo_description/meshes/LFinger32.dae" scale="1 1 1"/>
-			</geometry>
-			<origin rpy="0 0 0" xyz="0 0 0"/>
-		</visual>
-		<collision>
-			<geometry>
-				<mesh filename="package://romeo_description/meshes/LFinger32_0.10.stl" scale="1 1 1"/>
+				<mesh filename="package://romeo_description_mc/meshes/LFinger32.dae" scale="1 1 1"/>
+			</geometry>
+			<origin rpy="0 0 0" xyz="0 0 0"/>
+		</visual>
+		<collision>
+			<geometry>
+				<mesh filename="package://romeo_description_mc/meshes/LFinger32_0.10.stl" scale="1 1 1"/>
 			</geometry>
 			<origin rpy="0 0 0" xyz="0 0 0"/>
@@ -161,11 +161,11 @@
 		<visual>
 			<geometry>
-				<mesh filename="package://romeo_description/meshes/LThumb3.dae" scale="1 1 1"/>
-			</geometry>
-			<origin rpy="0 0 0" xyz="0 0 0"/>
-		</visual>
-		<collision>
-			<geometry>
-				<mesh filename="package://romeo_description/meshes/LThumb3_0.10.stl" scale="1 1 1"/>
+				<mesh filename="package://romeo_description_mc/meshes/LThumb3.dae" scale="1 1 1"/>
+			</geometry>
+			<origin rpy="0 0 0" xyz="0 0 0"/>
+		</visual>
+		<collision>
+			<geometry>
+				<mesh filename="package://romeo_description_mc/meshes/LThumb3_0.10.stl" scale="1 1 1"/>
 			</geometry>
 			<origin rpy="0 0 0" xyz="0 0 0"/>
@@ -175,11 +175,11 @@
 		<visual>
 			<geometry>
-				<mesh filename="package://romeo_description/meshes/HeadRoll.dae" scale="1 1 1"/>
-			</geometry>
-			<origin rpy="0 0 0" xyz="0 0 0"/>
-		</visual>
-		<collision>
-			<geometry>
-				<mesh filename="package://romeo_description/meshes/HeadRoll_0.10.stl" scale="1 1 1"/>
+				<mesh filename="package://romeo_description_mc/meshes/HeadRoll.dae" scale="1 1 1"/>
+			</geometry>
+			<origin rpy="0 0 0" xyz="0 0 0"/>
+		</visual>
+		<collision>
+			<geometry>
+				<mesh filename="package://romeo_description_mc/meshes/HeadRoll_0.10.stl" scale="1 1 1"/>
 			</geometry>
 			<origin rpy="0 0 0" xyz="0 0 0"/>
@@ -189,11 +189,11 @@
 		<visual>
 			<geometry>
-				<mesh filename="package://romeo_description/meshes/LThumb1.dae" scale="1 1 1"/>
-			</geometry>
-			<origin rpy="0 0 0" xyz="0 0 0"/>
-		</visual>
-		<collision>
-			<geometry>
-				<mesh filename="package://romeo_description/meshes/LThumb1_0.10.stl" scale="1 1 1"/>
+				<mesh filename="package://romeo_description_mc/meshes/LThumb1.dae" scale="1 1 1"/>
+			</geometry>
+			<origin rpy="0 0 0" xyz="0 0 0"/>
+		</visual>
+		<collision>
+			<geometry>
+				<mesh filename="package://romeo_description_mc/meshes/LThumb1_0.10.stl" scale="1 1 1"/>
 			</geometry>
 			<origin rpy="0 0 0" xyz="0 0 0"/>
@@ -203,11 +203,11 @@
 		<visual>
 			<geometry>
-				<mesh filename="package://romeo_description/meshes/LFinger11.dae" scale="1 1 1"/>
-			</geometry>
-			<origin rpy="0 0 0" xyz="0 0 0"/>
-		</visual>
-		<collision>
-			<geometry>
-				<mesh filename="package://romeo_description/meshes/LFinger11_0.10.stl" scale="1 1 1"/>
+				<mesh filename="package://romeo_description_mc/meshes/LFinger11.dae" scale="1 1 1"/>
+			</geometry>
+			<origin rpy="0 0 0" xyz="0 0 0"/>
+		</visual>
+		<collision>
+			<geometry>
+				<mesh filename="package://romeo_description_mc/meshes/LFinger11_0.10.stl" scale="1 1 1"/>
 			</geometry>
 			<origin rpy="0 0 0" xyz="0 0 0"/>
@@ -217,11 +217,11 @@
 		<visual>
 			<geometry>
-				<mesh filename="package://romeo_description/meshes/RFinger22.dae" scale="1 1 1"/>
-			</geometry>
-			<origin rpy="0 0 0" xyz="0 0 0"/>
-		</visual>
-		<collision>
-			<geometry>
-				<mesh filename="package://romeo_description/meshes/RFinger22_0.10.stl" scale="1 1 1"/>
+				<mesh filename="package://romeo_description_mc/meshes/RFinger22.dae" scale="1 1 1"/>
+			</geometry>
+			<origin rpy="0 0 0" xyz="0 0 0"/>
+		</visual>
+		<collision>
+			<geometry>
+				<mesh filename="package://romeo_description_mc/meshes/RFinger22_0.10.stl" scale="1 1 1"/>
 			</geometry>
 			<origin rpy="0 0 0" xyz="0 0 0"/>
@@ -231,11 +231,11 @@
 		<visual>
 			<geometry>
-				<mesh filename="package://romeo_description/meshes/LFinger22.dae" scale="1 1 1"/>
-			</geometry>
-			<origin rpy="0 0 0" xyz="0 0 0"/>
-		</visual>
-		<collision>
-			<geometry>
-				<mesh filename="package://romeo_description/meshes/LFinger22_0.10.stl" scale="1 1 1"/>
+				<mesh filename="package://romeo_description_mc/meshes/LFinger22.dae" scale="1 1 1"/>
+			</geometry>
+			<origin rpy="0 0 0" xyz="0 0 0"/>
+		</visual>
+		<collision>
+			<geometry>
+				<mesh filename="package://romeo_description_mc/meshes/LFinger22_0.10.stl" scale="1 1 1"/>
 			</geometry>
 			<origin rpy="0 0 0" xyz="0 0 0"/>
@@ -245,11 +245,11 @@
 		<visual>
 			<geometry>
-				<mesh filename="package://romeo_description/meshes/RFinger21.dae" scale="1 1 1"/>
-			</geometry>
-			<origin rpy="0 0 0" xyz="0 0 0"/>
-		</visual>
-		<collision>
-			<geometry>
-				<mesh filename="package://romeo_description/meshes/RFinger21_0.10.stl" scale="1 1 1"/>
+				<mesh filename="package://romeo_description_mc/meshes/RFinger21.dae" scale="1 1 1"/>
+			</geometry>
+			<origin rpy="0 0 0" xyz="0 0 0"/>
+		</visual>
+		<collision>
+			<geometry>
+				<mesh filename="package://romeo_description_mc/meshes/RFinger21_0.10.stl" scale="1 1 1"/>
 			</geometry>
 			<origin rpy="0 0 0" xyz="0 0 0"/>
@@ -259,11 +259,11 @@
 		<visual>
 			<geometry>
-				<mesh filename="package://romeo_description/meshes/RShoulderYaw.dae" scale="1 1 1"/>
-			</geometry>
-			<origin rpy="0 0 0" xyz="0 0 0"/>
-		</visual>
-		<collision>
-			<geometry>
-				<mesh filename="package://romeo_description/meshes/RShoulderYaw_0.10.stl" scale="1 1 1"/>
+				<mesh filename="package://romeo_description_mc/meshes/RShoulderYaw.dae" scale="1 1 1"/>
+			</geometry>
+			<origin rpy="0 0 0" xyz="0 0 0"/>
+		</visual>
+		<collision>
+			<geometry>
+				<mesh filename="package://romeo_description_mc/meshes/RShoulderYaw_0.10.stl" scale="1 1 1"/>
 			</geometry>
 			<origin rpy="0 0 0" xyz="0 0 0"/>
@@ -273,11 +273,11 @@
 		<visual>
 			<geometry>
-				<mesh filename="package://romeo_description/meshes/LWristRoll.dae" scale="1 1 1"/>
-			</geometry>
-			<origin rpy="0 0 0" xyz="0 0 0"/>
-		</visual>
-		<collision>
-			<geometry>
-				<mesh filename="package://romeo_description/meshes/LWristRoll_0.10.stl" scale="1 1 1"/>
+				<mesh filename="package://romeo_description_mc/meshes/LWristRoll.dae" scale="1 1 1"/>
+			</geometry>
+			<origin rpy="0 0 0" xyz="0 0 0"/>
+		</visual>
+		<collision>
+			<geometry>
+				<mesh filename="package://romeo_description_mc/meshes/LWristRoll_0.10.stl" scale="1 1 1"/>
 			</geometry>
 			<origin rpy="0 0 0" xyz="0 0 0"/>
@@ -287,11 +287,11 @@
 		<visual>
 			<geometry>
-				<mesh filename="package://romeo_description/meshes/RThumb1.dae" scale="1 1 1"/>
-			</geometry>
-			<origin rpy="0 0 0" xyz="0 0 0"/>
-		</visual>
-		<collision>
-			<geometry>
-				<mesh filename="package://romeo_description/meshes/RThumb1_0.10.stl" scale="1 1 1"/>
+				<mesh filename="package://romeo_description_mc/meshes/RThumb1.dae" scale="1 1 1"/>
+			</geometry>
+			<origin rpy="0 0 0" xyz="0 0 0"/>
+		</visual>
+		<collision>
+			<geometry>
+				<mesh filename="package://romeo_description_mc/meshes/RThumb1_0.10.stl" scale="1 1 1"/>
 			</geometry>
 			<origin rpy="0 0 0" xyz="0 0 0"/>
@@ -301,11 +301,11 @@
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