Commit message: Added intertial values for the eyes (from ufficial repo https://github.com/ros-aldebaran/romeo_robot/pull/13/commits/4a92d08096109cb7893767f2f0c8ca40cc845d59)

File: romeo_description_mc/urdf/romeo_eyes.xacro (robot description, xacro)
@@ -14,6 +14,6 @@
 		<inertial>
 			<mass value="0.01"/>
-			<inertia ixx="0" ixy="0" ixz="0" iyy="0" iyz="0" izz="0"/>
-			<origin rpy="0 0 0" xyz="0 0 0"/>
+            <inertia ixx="1e-09" ixy="0" ixz="0" iyy="1e-09" iyz="0" izz="1e-09" />
+			<origin rpy="0 -0 1.5708" xyz="0 0 0"/>
 		</inertial>
 	</link>
@@ -28,6 +28,6 @@
 		<inertial>
 			<mass value="0.01"/>
-			<inertia ixx="0" ixy="0" ixz="0" iyy="0" iyz="0" izz="0"/>
-			<origin rpy="0 0 0" xyz="0 0 0"/>
+			<inertia ixx="1e-09" ixy="0" ixz="0" iyy="1e-09" iyz="0" izz="1e-09" />
+     		<origin rpy="1.5708 -0 -3.14159" xyz="0 0 0"/>
 		</inertial>
 		<xacro:insert_visu_LEye/>
@@ -43,6 +43,6 @@
 		<inertial>
 			<mass value="0.01"/>
-			<inertia ixx="0" ixy="0" ixz="0" iyy="0" iyz="0" izz="0"/>
-			<origin rpy="0 0 0" xyz="0 0 0"/>
+			<inertia ixx="1e-09" ixy="0" ixz="0" iyy="1e-09" iyz="0" izz="1e-09" />
+ 			<origin rpy="0 -0 1.5708" xyz="0 0 0"/>
 		</inertial>
 	</link>
@@ -57,6 +57,6 @@
 		<inertial>
 			<mass value="0.01"/>
-			<inertia ixx="0" ixy="0" ixz="0" iyy="0" iyz="0" izz="0"/>
-			<origin rpy="0 0 0" xyz="0 0 0"/>
+			<inertia ixx="1e-09" ixy="0" ixz="0" iyy="1e-09" iyz="0" izz="1e-09" />
+ 			<origin rpy="1.5708 -0 -3.14159" xyz="0 0 0"/>
 		</inertial>
 		<xacro:insert_visu_REye/>
